Commit message: have end position match sva

File: arm/lite6.urdf (robot description, URDF)
Before this commit: robot UF_ROBOT, 8 links, 7 joints
Joints:
- joint joint6: origin xyz=0 0.0625 0 rpy=-1.5708 0 0 -> xyz=0 0.0625 0 rpy=-1.5708 3.14159265359 0

File: arm/xarm6.urdf (robot description, URDF)
Before this commit: robot UF_ROBOT, 9 links, 8 joints
Joints:
- joint joint6: origin xyz=0.076 0.097 0 rpy=-1.5708 0 0 -> xyz=0.076 0.097 0 rpy=-1.5708 3.14159265359 0

File: arm/xarm7.urdf (robot description, URDF)
Before this commit: robot UF_ROBOT, 9 links, 8 joints
Joints:
- joint joint7: origin xyz=0.076 0.097 0 rpy=-1.5708 0 0 -> xyz=0.076 0.097 0 rpy=-1.5708 3.14159265359 0
