Commit message: update

File: arm/lite6.urdf (robot description, URDF)
Before this commit: robot UF_ROBOT, 8 links, 7 joints
Links:
- added link link_eef
- link link6: geometry 
Joints:
- added joint joint_eef: type fixed, parent link6, child link_eef, origin xyz=0 0 0 rpy=0 0 0

File: arm/uf850.urdf (robot description, URDF)
Before this commit: robot UF_ROBOT, 8 links, 6 joints
Links:
- added link link_eef
- link link6: geometry 
Joints:
- added joint joint_eef: type fixed, parent link6, child link_eef, origin xyz=0 0 0 rpy=0 0 0

File: arm/xarm6_1305.urdf (robot description, URDF)
Before this commit: robot UF_ROBOT, 9 links, 8 joints
Links:
- link link6: geometry 

File: arm/xarm7.urdf (robot description, URDF)
Before this commit: robot UF_ROBOT, 9 links, 8 joints
Links:
- added link link_eef
Joints:
- added joint joint_eef: type fixed, parent link7, child link_eef, origin xyz=0 0 0 rpy=0 0 0

Commit message: support last mesh

File: arm/lite6.urdf (robot description, URDF)
Before this commit: robot UF_ROBOT, 9 links, 8 joints
Links:
- link link6: geometry collision mesh filename=package://description/meshes/lite6meshes/link6.stl

File: arm/uf850.urdf (robot description, URDF)
Before this commit: robot UF_ROBOT, 9 links, 7 joints
Links:
- link link6: geometry collision mesh filename=package://description/meshes/uf850meshes/link6.stl

File: arm/xarm6_1305.urdf (robot description, URDF)
Before this commit: robot UF_ROBOT, 9 links, 8 joints
Links:
- link link6: geometry collision mesh filename=package://description/meshes/xarm6_1305meshes/link6.stl

Commit message: comments

File: arm/lite6.urdf (robot description, URDF)
Before this commit: robot UF_ROBOT, 9 links, 8 joints
Links:
- removed link link_eef
Joints:
- removed joint joint_eef

File: arm/uf850.urdf (robot description, URDF)
Before this commit: robot UF_ROBOT, 9 links, 7 joints
Links:
- removed link link_eef
Joints:
- removed joint joint_eef

File: arm/xarm7.urdf (robot description, URDF)
Before this commit: robot UF_ROBOT, 10 links, 9 joints
Links:
- removed link link_eef
Joints:
- removed joint joint_eef
